Commit message: IMU shows in rviz

File: description/urdf/cybertruck.urdf.xacro (robot description, xacro)
@@ -32,5 +32,15 @@
     <xacro:include filename="$(find description)/urdf/wheels.urdf.xacro"/>
     <!-- LIDAR (also used for IMU) -->
-    <link name="scan_link"/>
+    <link name="scan_link">
+        <visual>
+            <origin xyz="0 0 0" rpy="0 0 0" />
+            <geometry>
+                <box size="0.1 0.1 0.1" />
+            </geometry>
+            <material name="Cyan">
+                <color rgba="0 1.0 1.0 1.0"/>
+            </material>
+        </visual>
+    </link>
     <joint name="scan_joint" type="fixed">
         <parent link="body_link"/>

File: description/urdf/plugins.gazebo.xacro (robot description, xacro)
@@ -45,7 +45,8 @@
             <plugin filename="libgazebo_ros_imu_sensor.so" name="imu_plugin">
                 <topicName>imu/data</topicName>
+                <!-- How come I don't need to say photon/imu/data ^^ there, below i listed out photon/scan_link instead of scan/link. I laso changed the reference from scan_link to photon/imu_link -->
                 <!-- Ask about topicName/ bodyName. Why do we do it all to the scan_link, but in caffeine they do it by scan_link/imu -->
-                <bodyName>scan_link</bodyName>
-                <frameName>scan_link</frameName>
+                <bodyName>photon/scan_link</bodyName>
+                <frameName>photon/scan_link</frameName>
                 <updateRateHZ>${imu_update_rate}</updateRateHZ>
                 <gaussianNoise>0.0</gaussianNoise>

Commit message: Added Visual boxes for both Lidar and IMU plugins

File: description/urdf/cybertruck.urdf.xacro (robot description, xacro)
@@ -31,10 +31,10 @@
     <!-- Wheels -->
     <xacro:include filename="$(find description)/urdf/wheels.urdf.xacro"/>
-    <!-- LIDAR (also used for IMU) -->
-    <link name="scan_link">
+     <!-- LIDAR -->
+    <link name="lidar_link">
         <visual>
             <origin xyz="0 0 0" rpy="0 0 0" />
             <geometry>
-                <box size="0.1 0.1 0.1" />
+                <box size="0.03 0.03 0.03" />
             </geometry>
             <material name="Cyan">
@@ -43,8 +43,25 @@
         </visual>
     </link>
-    <joint name="scan_joint" type="fixed">
+    <joint name="lidar_joint" type="fixed">
         <parent link="body_link"/>
-        <child link="scan_link"/>
-        <origin xyz="0 ${fb_separation/2} ${-height_to_wheel}" rpy="0 0 0"/>
+        <child link="lidar_link"/>
+        <origin xyz="${fb_separation/2} 0 ${-height_to_wheel/2}" rpy="0 0 0"/>
+    </joint>
+     <!-- IMU -->
+    <link name="imu_link">
+        <visual>
+            <origin xyz="0 0 0" rpy="0 0 0" />
+            <geometry>
+                <box size="0.03 0.03 0.03" />
+            </geometry>
+            <material name="Cyan">
+                <color rgba="0 0.0 1.0 1.0"/>
+            </material>
+        </visual>
+    </link>
+    <joint name="imu_joint" type="fixed">
+        <parent link="body_link"/>
+        <child link="imu_link"/>
+        <origin xyz="0 0 ${-height_to_wheel}" rpy="0 0 0"/>
     </joint>
 </robot>

File: description/urdf/plugins.gazebo.xacro (robot description, xacro)
@@ -4,5 +4,5 @@
     <xacro:include filename="$(find description)/urdf/constants.xacro"/>
     <!-- LIDAR -->
-    <gazebo reference="scan_link">
+    <gazebo reference="lidar_link">
         <sensor type="ray" name="gpu_hokuyo_sensor">
             <pose>0 0 0 0 0 0</pose>
@@ -32,10 +32,10 @@
             <plugin name="gazebo_ros_hokuyo_controller" filename="libgazebo_ros_laser.so">
                 <topicName>scan</topicName>
-                <frameName>scan_link</frameName>
+                <frameName>lidar_link</frameName>
             </plugin>
         </sensor>
     </gazebo>
     <!-- IMU -->
-    <gazebo reference="scan_link">
+    <gazebo reference="imu_link">
         <gravity>true</gravity>
         <sensor name="imu_sensor" type="imu">
@@ -45,8 +45,6 @@
             <plugin filename="libgazebo_ros_imu_sensor.so" name="imu_plugin">
                 <topicName>imu/data</topicName>
-                <!-- How come I don't need to say photon/imu/data ^^ there, below i listed out photon/scan_link instead of scan/link. I laso changed the reference from scan_link to photon/imu_link -->
-                <!-- Ask about topicName/ bodyName. Why do we do it all to the scan_link, but in caffeine they do it by scan_link/imu -->
-                <bodyName>photon/scan_link</bodyName>
-                <frameName>photon/scan_link</frameName>
+                <bodyName>photon/imu_link</bodyName>
+                <frameName>photon/imu_link</frameName>
                 <updateRateHZ>${imu_update_rate}</updateRateHZ>
                 <gaussianNoise>0.0</gaussianNoise>
