Commit message: Created a plugins.gazebo.xacro, added lidar joints in cypertruck.urdf.xacro. Not tested.

File: description/urdf/constants.xacro (robot description, xacro)
@@ -5,3 +5,4 @@
     <xacro:property name="lr_separation" value="0.304"/>
     <xacro:property name="height_to_wheel" value="-0.1135"/>
+    <xacro:property name="front_wheel" value="${fb_separation/2}"/>
 </robot>

File: description/urdf/cybertruck.urdf.xacro (robot description, xacro)
@@ -4,4 +4,5 @@
     <xacro:include filename="$(find description)/urdf/constants.xacro"/>
     <xacro:include filename="$(find description)/urdf/inertias.xacro"/>
+    <!-- <xacro:include filename="$(find description)/urdf/plugins.gazebo.xacro"/> -->
     <link name="base_link"/>
     <!-- Body -->
@@ -30,3 +31,10 @@
     <!-- Wheels -->
     <xacro:include filename="$(find description)/urdf/wheels.urdf.xacro"/>
+    <!-- LIDAR (also used for IMU) -->
+    <link name="scan_link"/>
+    <joint name="scan_joint" type="fixed">
+        <parent link="body_link"/>
+        <child link="scan_link"/>
+        <origin xyz="0 ${front_wheel} ${-height_to_wheel}" rpy="0 0 0"/>
+    </joint>
 </robot>

Commit message: formatting changes

File: description/urdf/constants.xacro (robot description, xacro)
@@ -3,23 +3,9 @@
     <!-- Body properties -->
     <xacro:property name="body_mass" value="1.33"/>
-    <xacro:property name="body_ixx" value="0.00563"/>
-    <xacro:property name="body_ixy" value="0"/>
-    <xacro:property name="body_ixz" value="0.00003"/>
-    <xacro:property name="body_iyy" value="0.01814"/>
-    <xacro:property name="body_iyz" value="0"/>
-    <xacro:property name="body_izz" value="0.02119"/>
     <!-- Wheels properties -->
     <xacro:property name="wheel_mass" value="0.125"/>
-    <xacro:property name="wheel_ixx" value="0.000256"/>
-    <xacro:property name="wheel_ixy" value="0"/>
-    <xacro:property name="wheel_ixz" value="0"/>
-    <xacro:property name="wheel_iyy" value="0.000296"/>
-    <xacro:property name="wheel_iyz" value="0"/>
-    <xacro:property name="wheel_izz" value="0.000256"/>
     <!-- Distances from Body to Wheels -->
-    <xacro:property name="front_wheel" value="0.143"/>
-    <xacro:property name="back_wheel" value="${0.143-0.286}"/>
-    <xacro:property name="right_wheel" value="-0.15205"/>
-    <xacro:property name="left_wheel" value="0.15205"/>
+    <xacro:property name="fb_separation" value="0.286"/>
+    <xacro:property name="lr_separation" value="0.304"/>
     <xacro:property name="height_to_wheel" value="-0.1135"/>
 </robot>

File: description/urdf/cybertruck.urdf.xacro (robot description, xacro)
@@ -3,4 +3,5 @@
     <!-- Includes -->
     <xacro:include filename="$(find description)/urdf/constants.xacro"/>
+    <xacro:include filename="$(find description)/urdf/inertias.xacro"/>
     <link name="base_link"/>
     <!-- Body -->
@@ -20,6 +21,5 @@
         <inertial>
             <mass value="${body_mass}"/>
-            <inertia ixx="${body_ixx}"  ixy="${body_ixy}"  ixz="${body_ixz}"
-                        iyy="${body_iyy}" iyz="${body_iyz}" izz="${body_izz}" />
+            <xacro:body_inertia/>
         </inertial>
     </link>

File: description/urdf/wheels.urdf.xacro (robot description, xacro)
@@ -3,4 +3,5 @@
     <!-- Includes -->
     <xacro:include filename="$(find description)/urdf/constants.xacro"/>
+    <xacro:include filename="$(find description)/urdf/inertias.xacro"/>
     <!-- Wheel macro -->
     <xacro:macro name="Wheel" params="fb lr">
@@ -20,7 +21,6 @@
             </collision>
             <inertial>
-            <mass value="${wheel_mass}"/>
-            <inertia ixx="${wheel_ixx}"  ixy="${wheel_ixy}"  ixz="${wheel_ixz}"
-                        iyy="${wheel_iyy}" iyz="${wheel_iyz}" izz="${wheel_izz}" />
+                <mass value="${wheel_mass}"/>
+                <xacro:wheel_inertia/>
             </inertial>
         </link>
@@ -29,6 +29,6 @@
             <parent link="body_link"/>
             <child link="${fb}_${lr}_wheel_link"/>
-            <origin xyz="${front_wheel if fb == 'front' else back_wheel}
-                    ${left_wheel if lr == 'left' else right_wheel}
+            <origin xyz="${fb_separation/2 if fb == 'front' else -fb_separation/2}
+                    ${-lr_separation/2 if lr == 'left' else lr_separation/2}
                     ${height_to_wheel}" rpy="0 0 0"/>
             <axis xyz="0 1 0"/>

Commit message: editted inertia

File: description/urdf/constants.xacro (robot description, xacro)
@@ -1,8 +1,4 @@
 <?xml version="1.0"?>
 <robot name="constants" xmlns:xacro="http://ros.org/wiki/xacro">
-    <!-- Body properties -->
-    <xacro:property name="body_mass" value="1.33"/>
-    <!-- Wheels properties -->
-    <xacro:property name="wheel_mass" value="0.125"/>
     <!-- Distances from Body to Wheels -->
     <xacro:property name="fb_separation" value="0.286"/>

File: description/urdf/cybertruck.urdf.xacro (robot description, xacro)
@@ -20,5 +20,4 @@
         </collision>
         <inertial>
-            <mass value="${body_mass}"/>
             <xacro:body_inertia/>
         </inertial>

File: description/urdf/inertias.xacro (robot description, xacro)
@@ -3,16 +3,18 @@
     <!-- Body -->
     <xacro:macro name="body_inertia">
+        <mass value="1.33"/>
         <inertia
             ixx="1.33" ixy="0.00563" ixz="0.00003"
-            iyx="0.0000" iyy="0.01814" iyz="0.0000"
-            izx="0.0000" izy="0.0000" izz="0.02119"
+            iyy="0.01814" iyz="0.0000"
+            izz="0.02119"
         />
     </xacro:macro>
     <!-- Wheels -->
     <xacro:macro name="wheel_inertia">
+        <mass value="0.125"/>
         <inertia
             ixx="0.125" ixy="0.000256" ixz="0.0000"
-            iyx="0.0000" iyy="0.000296" iyz="0.0000"
-            izx="0.0000" izy="0.0000" izz="0.000256"
+            iyy="0.000296" iyz="0.0000"
+            izz="0.000256"
         />
     </xacro:macro>

File: description/urdf/wheels.urdf.xacro (robot description, xacro)
@@ -21,5 +21,4 @@
             </collision>
             <inertial>
-                <mass value="${wheel_mass}"/>
                 <xacro:wheel_inertia/>
             </inertial>

Commit message: Changed plugin file name and added constants to sensor

File: description/urdf/constants.xacro (robot description, xacro)
@@ -6,3 +6,8 @@
     <xacro:property name="height_to_wheel" value="-0.1135"/>
     <xacro:property name="front_wheel" value="${fb_separation/2}"/>
+    <!-- LIDAR -->
+    <xacro:property name="laser_update_rate" value="10"/>
+    <xacro:property name="laser_field_of_view" value="270"/>
+    <xacro:property name="laser_min_range" value="0.06"/>
+    <xacro:property name="laser_max_range" value="4.095"/>
 </robot>

File: description/urdf/cybertruck.urdf.xacro (robot description, xacro)
@@ -4,5 +4,5 @@
     <xacro:include filename="$(find description)/urdf/constants.xacro"/>
     <xacro:include filename="$(find description)/urdf/inertias.xacro"/>
-    <xacro:include filename="$(find description)/urdf/lidar_plugin.gazebo.xacro"/>
+    <xacro:include filename="$(find description)/urdf/plugins.gazebo.xacro"/>
     <link name="base_link"/>
     <!-- Body -->

File: description/urdf/plugins.gazebo.xacro (robot description, xacro)
@@ -2,5 +2,5 @@
 <robot name="plugins" xmlns:xacro="http://ros.org/wiki/xacro">
     <!-- Constants -->
-    <xacro:property name="laser_update_rate" value="10"/>
+    <xacro:include filename="$(find description)/urdf/constants.xacro"/>
     <!-- LIDAR -->
     <gazebo reference="scan_link">
@@ -9,5 +9,4 @@
             <!-- Set visualize to true for now -->
             <visualize>true</visualize>
-            <!-- Changed update rate from 30 to 10 -->
             <update_rate>${laser_update_rate}</update_rate>
             <ray>
@@ -16,12 +15,12 @@
                         <samples>1080</samples>
                         <resolution>1</resolution>
-                        <min_angle>${-0.5 * 270 * pi/180}</min_angle>
-                        <max_angle>${0.5 * 270 * pi/180}</max_angle>
+                        <min_angle>${-0.5*laser_field_of_view*pi/180}</min_angle>
+                        <max_angle>${0.5*laser_field_of_view*pi/180}</max_angle>
                     </horizontal>
                 </scan>
                 <range>
-                    <min>0.06</min>
-                    <max>4.095</max>
-                    <resolution>${0.36 * pi/180}</resolution>
+                    <min>${laser_min_range}</min>
+                    <max>${laser_max_range}</max>
+                    <resolution>${0.36* pi/180}</resolution>
                 </range>
                 <noise>

Commit message: Set visualize to false and other minor requested changes

File: description/urdf/constants.xacro (robot description, xacro)
@@ -5,6 +5,6 @@
     <xacro:property name="lr_separation" value="0.304"/>
     <xacro:property name="height_to_wheel" value="-0.1135"/>
-    <xacro:property name="front_wheel" value="${fb_separation/2}"/>
     <!-- LIDAR -->
+    <xacro:property name="laser_visualize" value="false"/>
     <xacro:property name="laser_update_rate" value="10"/>
     <xacro:property name="laser_field_of_view" value="270"/>

File: description/urdf/cybertruck.urdf.xacro (robot description, xacro)
@@ -36,5 +36,5 @@
         <parent link="body_link"/>
         <child link="scan_link"/>
-        <origin xyz="0 ${front_wheel} ${-height_to_wheel}" rpy="0 0 0"/>
+        <origin xyz="0 ${fb_separation/2} ${-height_to_wheel}" rpy="0 0 0"/>
     </joint>
 </robot>

File: description/urdf/plugins.gazebo.xacro (robot description, xacro)
@@ -7,6 +7,5 @@
         <sensor type="ray" name="gpu_hokuyo_sensor">
             <pose>0 0 0 0 0 0</pose>
-            <!-- Set visualize to true for now -->
-            <visualize>true</visualize>
+            <visualize>${laser_visualize}</visualize>
             <update_rate>${laser_update_rate}</update_rate>
             <ray>

Commit message: PHN2 - Simulate LIDAR (#12)
* Created a plugins.gazebo.xacro, added lidar joints in cypertruck.urdf.xacro. Not tested.

* Added Lidar Plugin. Simulates in Gazebo but not in rviz

* Changed plugin filename to lidar_plugin

* Set Lidar values as the same as Caffeine values

* Changed plugin file name and added constants to sensor

* Set visualize to false and other minor requested changes

* Added comment about missing actual lidar values

File: description/urdf/constants.xacro (robot description, xacro)
@@ -5,3 +5,9 @@
     <xacro:property name="lr_separation" value="0.304"/>
     <xacro:property name="height_to_wheel" value="-0.1135"/>
+    <!-- LIDAR -->
+    <xacro:property name="laser_visualize" value="false"/>
+    <xacro:property name="laser_update_rate" value="10"/>
+    <xacro:property name="laser_field_of_view" value="270"/>
+    <xacro:property name="laser_min_range" value="0.06"/>
+    <xacro:property name="laser_max_range" value="4.095"/>
 </robot>

File: description/urdf/cybertruck.urdf.xacro (robot description, xacro)
@@ -4,4 +4,5 @@
     <xacro:include filename="$(find description)/urdf/constants.xacro"/>
     <xacro:include filename="$(find description)/urdf/inertias.xacro"/>
+    <xacro:include filename="$(find description)/urdf/plugins.gazebo.xacro"/>
     <link name="base_link"/>
     <!-- Body -->
@@ -30,3 +31,10 @@
     <!-- Wheels -->
     <xacro:include filename="$(find description)/urdf/wheels.urdf.xacro"/>
+    <!-- LIDAR (also used for IMU) -->
+    <link name="scan_link"/>
+    <joint name="scan_joint" type="fixed">
+        <parent link="body_link"/>
+        <child link="scan_link"/>
+        <origin xyz="0 ${fb_separation/2} ${-height_to_wheel}" rpy="0 0 0"/>
+    </joint>
 </robot>

Commit message: Added IMU plugin with updated_rate constant

File: description/urdf/constants.xacro (robot description, xacro)
@@ -11,3 +11,5 @@
     <xacro:property name="laser_min_range" value="0.06"/>
     <xacro:property name="laser_max_range" value="4.095"/>
+    <!-- IMU -->
+    <xacro:property name="imu_update_rate" value="128"/>
 </robot>

File: description/urdf/plugins.gazebo.xacro (robot description, xacro)
@@ -36,3 +36,24 @@
         </sensor>
     </gazebo>
+    <!-- IMU -->
+    <gazebo reference="scan_link">
+        <gravity>true</gravity>
+        <sensor name="imu_sensor" type="imu">
+            <always_on>true</always_on>
+            <update_rate>${imu_update_rate}</update_rate>
+            <topic>__default_topic__</topic>
+            <plugin filename="libgazebo_ros_imu_sensor.so" name="imu_plugin">
+                <topicName>imu/data</topicName>
+                <!-- Ask about topicName/ bodyName. Why do we do it all to the scan_link, but in caffeine they do it by scan_link/imu -->
+                <bodyName>scan_link</bodyName>
+                <frameName>scan_link</frameName>
+                <updateRateHZ>${imu_update_rate}</updateRateHZ>
+                <gaussianNoise>0.0</gaussianNoise>
+                <xyzOffset>0 0 0</xyzOffset>
+                <rpyOffset>0 0 0</rpyOffset>
+                <initialOrientationAsReference>false</initialOrientationAsReference>
+            </plugin>
+            <pose>0 0 0 0 0 0</pose>
+        </sensor>
+    </gazebo>
 </robot>

Commit message: all files are in. code based on caffeine ZED camera. error when launching

File: description/urdf/constants.xacro (robot description, xacro)
@@ -11,3 +11,23 @@
     <xacro:property name="laser_min_range" value="0.06"/>
     <xacro:property name="laser_max_range" value="4.095"/>
+        <xacro:property name="camera_mass" value="0.1587573"/>
+    <xacro:property name="camera_length" value="0.175"/>
+    <xacro:property name="camera_width" value="0.03"/>
+    <xacro:property name="camera_height" value="0.033"/>
+    <xacro:property name="camera_pitch" value="${15 * pi/180}"/>
+    <!-- Camera image height/width corresponds to image size for 60Hz refresh-->
+    <xacro:property name="image_refresh" value="60"/>
+    <xacro:property name="image_width" value="3840"/>
+    <xacro:property name="image_height" value="1080"/>
+    <xacro:property name="image_format" value="R8G8B8"/>
+    <xacro:property name="image_hfov" value="${90 * pi/180}"/>
+    <xacro:property name="name" value="camera/camera_node"/>
+    <xacro:property name="always_on" value="true"/>
+    <xacro:property name="update_rate" value="0"/>
+    <xacro:property name="image_topicName" value="image_raw_color"/>
+    <xacro:property name="image_info_topicName" value="camera_info"/>
+    <xacro:property name="depth_topicName" value="depth/image_raw"/>
+    <xacro:property name="depth_info_topicName" value="depth/camera_info"/>
+    <xacro:property name="depth_points_topicName" value="depth/points"/>
+    <xacro:property name="frameName" value="zed_camera_link_optical"/>
 </robot>

File: description/urdf/cybertruck.urdf.xacro (robot description, xacro)
@@ -38,3 +38,27 @@
         <origin xyz="0 ${fb_separation/2} ${-height_to_wheel}" rpy="0 0 0"/>
     </joint>
+    <!-- ZED Camera -->
+    <link name="${tf_prefix}/camera_link">
+        <visual>
+            <origin xyz="0 0 0" rpy="0 0 0"/>
+            <geometry>
+            <box size="${camera_width} ${camera_length} ${camera_height}"/>
+            </geometry>
+        </visual>
+        <collision>
+            <origin xyz="0 0 0" rpy="0 0 0"/>
+            <geometry>
+                <box size="${camera_width} ${camera_length} ${camera_height}"/>
+            </geometry>
+        </collision>
+        <inertial>
+            <xacro:box_inertia mass="${camera_mass}" length="${camera_length}" width="${camera_width}" height="${camera_height}"/>
+            <mass value="${camera_mass}"/>
+        </inertial>
+    </link>
+    <joint name="${tf_prefix}/camera_joint" type="fixed">
+        <origin xyz="${stand_length/2 - camera_width} 0 ${camera_height / 2.0}" rpy="0 ${camera_pitch} 0"/>
+        <parent link="${tf_prefix}/stand_link"/>
+        <child link="${tf_prefix}/camera_link"/>
+    </joint>
 </robot>

File: description/urdf/plugins.gazebo.xacro (robot description, xacro)
@@ -36,3 +36,53 @@
         </sensor>
     </gazebo>
+<!--Stereo Camera-->
+    <!-- Gazebo multicamera plugin -->
+    <gazebo reference="${tf_prefix}/camera_link">
+        <sensor type="multicamera" name="stereo_camera">
+            <update_rate>${image_refresh}</update_rate>
+            <camera name="left">
+            <horizontal_fov>${image_hfov}</horizontal_fov>
+            <image>
+                <width>${image_width}</width>
+                <height>${image_height}</height>
+                <format>${image_format}</format>
+            </image>
+            <clip>
+                <near>0.02</near>
+                <far>300</far>
+            </clip>
+            </camera>
+            <camera name="right">
+            <pose>0 ${-camera_length} 0 0 0 0</pose>
+            <horizontal_fov>${image_hfov}</horizontal_fov>
+            <image>
+                <width>${image_width}</width>
+                <height>${image_height}</height>
+                <format>${image_format}</format>
+            </image>
+            <clip>
+                <near>0.02</near>
+                <far>300</far>
+            </clip>
+            </camera>
+            <plugin name="stereo_camera_controller" filename="libgazebo_ros_multicamera.so">
+                <cameraName>${name}</cameraName>
+                <alwaysOn>${always_on}</alwaysOn>
+                <updateRate>${update_rate}</updateRate>
+                <imageTopicName>${image_topicName}</imageTopicName>
+                <cameraInfoTopicName>${image_info_topicName}</cameraInfoTopicName>
+                <depthImageTopicName>${depth_topicName}</depthImageTopicName>
+                <depthImageInfoTopicName>${depth_info_topicName}</depthImageInfoTopicName>
+                <pointCloudTopicName>${depth_points_topicName}</pointCloudTopicName>
+                <frameName>${tf_prefix}/${frameName}</frameName>
+                <hackBaseline>${camera_length}</hackBaseline>
+                <!-- TODO: Get distortion parameters from real camera -->
+                <distortionK1>0.0</distortionK1>
+                <distortionK2>0.0</distortionK2>
+                <distortionK3>0.0</distortionK3>
+                <distortionT1>0.0</distortionT1>
+                <distortionT2>0.0</distortionT2>
+            </plugin>
+        </sensor>
+    </gazebo>
 </robot>

Commit message: added ackermann steering controller and corresponding urdf and launch files

File: description/urdf/constants.xacro (robot description, xacro)
@@ -5,9 +5,12 @@
     <xacro:property name="lr_separation" value="0.304"/>
     <xacro:property name="height_to_wheel" value="-0.1135"/>
-    <!-- LIDAR -->
-    <xacro:property name="laser_visualize" value="false"/>
-    <xacro:property name="laser_update_rate" value="10"/>
-    <xacro:property name="laser_field_of_view" value="270"/>
-    <xacro:property name="laser_min_range" value="0.06"/>
-    <xacro:property name="laser_max_range" value="4.095"/>
+    <!-- Wheel dimensions -->
+    <xacro:property name="wheel_radius" value="0.0635"/>
+    <xacro:property name="thickness" value="0.1016"/>
+    <!-- Steer dimensions -->
+    <xacro:property name="steer_radius" value="0.05" />
+    <xacro:property name="steer_thickness" value="0.02" />
+    <xacro:property name="steer_effort"   value="10.0"/>
+    <xacro:property name="steer_velocity" value="5.0"/>
+    <xacro:property name="deg_to_rad" value="0.01745329251994329577"/>
 </robot>

Commit message: PHN8 - Created launch files to build custom worlds in gazebo  (#10)
* created remote branch for issue #8

* added files from 2019Resources repository, need to start working on getting the worlds to work in gazebo

* added boilerplate from sim_tutorial

* Set up all the models in their correct folders and started working on world files for each world. Have not tested to see if world works yet

* Addedlaunch files for the worlds to be able to build them in Gazebo.

* Addedthe sdf, material, and config files. Added to gazebo model folder. It still does not spawn

* Run install_sh files. Sumo Ring works

* got gazebo to recognize that models should be imported from circuits directory, but the model doesn't show up, only a dark grey rectangle does.

* Able to see the circuit race world in Gazebo using the .material file. Need to use stl into .sdf

* Comment to test push

* Changed world files, and the robot spawned in GAzebo. Done through sdf files and .materials

* deleted things pertaining to sumo

* formattin everything + deleted more sumo stuff

* fomatting changes and deletions of unnecessary files

* made changes as instructed by Erick. Started working on a unified iaarc.world files which allows for choosing world based on arguments. So far not crashing, but not loading either.

* added package.xml for it to load worlds properly. Next step is to load circuit and drag_race to scale.

* resized circuit and drag race to be approximately equal to the size specified within the rules booklet

* renamed files, added newlines, deleted redundant files

Co-authored-by: EsteBran <tawseefhanif@gmail.com>
Co-authored-by: Paula Santas Rodriguez <psantasr>

File: description/urdf/constants.xacro (robot description, xacro)
@@ -1,4 +1,14 @@
 <?xml version="1.0"?>
 <robot name="constants" xmlns:xacro="http://ros.org/wiki/xacro">
+    <!-- Body properties -->
+    <xacro:property name="body_mass" value="2.5"/>
+    <xacro:property name="body_length" value="0.14"/>
+    <xacro:property name="body_width" value="0.05"/>
+    <xacro:property name="body_height" value="0.04"/>
+    <!-- Wheels properties -->
+    <xacro:property name="wheel_mass" value="0.05"/>
+    <xacro:property name="wheel_radius" value="0.01"/>
+    <xacro:property name="wheel_width" value="0.006"/>
+    <xacro:property name="wheel_separation" value="0.047"/>
     <!-- Distances from Body to Wheels -->
     <xacro:property name="fb_separation" value="0.286"/>

Commit message: push routine

File: description/urdf/constants.xacro (robot description, xacro)
@@ -26,6 +26,6 @@
     <xacro:property name="update_rate" value="0"/>
     <xacro:property name="image_topicName" value="image_raw_color"/>
-    <xacro:property name="image_info_topicName" value="camera_info"/>
-    <xacro:property name="depth_topicName" value="depth/image_raw"/>
+    <!--xacro:property name="image_info_topicName" value="camera_info"/-->
+    <!--xacro:property name="depth_topicName" value="depth/image_raw"/-->
     <xacro:property name="depth_info_topicName" value="depth/camera_info"/>
     <xacro:property name="depth_points_topicName" value="depth/points"/>
