Commit message: PHN3 - Simulate IMU (#14)
* Added IMU plugin with updated_rate constant

* IMU shows in rviz

* Added Visual boxes for both Lidar and IMU plugins

File: description/urdf/constants.xacro (robot description, xacro)
@@ -21,3 +21,5 @@
     <xacro:property name="laser_min_range" value="0.06"/>
     <xacro:property name="laser_max_range" value="4.095"/>
+    <!-- IMU -->
+    <xacro:property name="imu_update_rate" value="128"/>
 </robot>

File: description/urdf/cybertruck.urdf.xacro (robot description, xacro)
@@ -31,10 +31,37 @@
     <!-- Wheels -->
     <xacro:include filename="$(find description)/urdf/wheels.urdf.xacro"/>
-    <!-- LIDAR (also used for IMU) -->
-    <link name="scan_link"/>
-    <joint name="scan_joint" type="fixed">
+     <!-- LIDAR -->
+    <link name="lidar_link">
+        <visual>
+            <origin xyz="0 0 0" rpy="0 0 0" />
+            <geometry>
+                <box size="0.03 0.03 0.03" />
+            </geometry>
+            <material name="Cyan">
+                <color rgba="0 1.0 1.0 1.0"/>
+            </material>
+        </visual>
+    </link>
+    <joint name="lidar_joint" type="fixed">
         <parent link="body_link"/>
-        <child link="scan_link"/>
-        <origin xyz="0 ${fb_separation/2} ${-height_to_wheel}" rpy="0 0 0"/>
+        <child link="lidar_link"/>
+        <origin xyz="${fb_separation/2} 0 ${-height_to_wheel/2}" rpy="0 0 0"/>
+    </joint>
+     <!-- IMU -->
+    <link name="imu_link">
+        <visual>
+            <origin xyz="0 0 0" rpy="0 0 0" />
+            <geometry>
+                <box size="0.03 0.03 0.03" />
+            </geometry>
+            <material name="Cyan">
+                <color rgba="0 0.0 1.0 1.0"/>
+            </material>
+        </visual>
+    </link>
+    <joint name="imu_joint" type="fixed">
+        <parent link="body_link"/>
+        <child link="imu_link"/>
+        <origin xyz="0 0 ${-height_to_wheel}" rpy="0 0 0"/>
     </joint>
 </robot>

File: description/urdf/plugins.gazebo.xacro (robot description, xacro)
@@ -4,5 +4,5 @@
     <xacro:include filename="$(find description)/urdf/constants.xacro"/>
     <!-- LIDAR -->
-    <gazebo reference="scan_link">
+    <gazebo reference="lidar_link">
         <sensor type="ray" name="gpu_hokuyo_sensor">
             <pose>0 0 0 0 0 0</pose>
@@ -32,7 +32,27 @@
             <plugin name="gazebo_ros_hokuyo_controller" filename="libgazebo_ros_laser.so">
                 <topicName>scan</topicName>
-                <frameName>scan_link</frameName>
+                <frameName>lidar_link</frameName>
             </plugin>
         </sensor>
     </gazebo>
+    <!-- IMU -->
+    <gazebo reference="imu_link">
+        <gravity>true</gravity>
+        <sensor name="imu_sensor" type="imu">
+            <always_on>true</always_on>
+            <update_rate>${imu_update_rate}</update_rate>
+            <topic>__default_topic__</topic>
+            <plugin filename="libgazebo_ros_imu_sensor.so" name="imu_plugin">
+                <topicName>imu/data</topicName>
+                <bodyName>photon/imu_link</bodyName>
+                <frameName>photon/imu_link</frameName>
+                <updateRateHZ>${imu_update_rate}</updateRateHZ>
+                <gaussianNoise>0.0</gaussianNoise>
+                <xyzOffset>0 0 0</xyzOffset>
+                <rpyOffset>0 0 0</rpyOffset>
+                <initialOrientationAsReference>false</initialOrientationAsReference>
+            </plugin>
+            <pose>0 0 0 0 0 0</pose>
+        </sensor>
+    </gazebo>
 </robot>

Commit message: changes allows for launching camera not there

File: description/urdf/constants.xacro (robot description, xacro)
@@ -37,5 +37,5 @@
     <xacro:property name="image_topicName" value="image_raw_color"/>
     <xacro:property name="image_info_topicName" value="camera_info"/>
-    <!--xacro:property name="depth_topicName" value="depth/image_raw"/-->
+    <xacro:property name="depth_topicName" value="depth/image_raw"/>
     <xacro:property name="depth_info_topicName" value="depth/camera_info"/>
     <xacro:property name="depth_points_topicName" value="depth/points"/>

File: description/urdf/cybertruck.urdf.xacro (robot description, xacro)
@@ -66,5 +66,5 @@
     </joint>
     <!-- ZED Camera -->
-    <link name="${tf_prefix}/camera_link">
+    <link name="camera_link">
         <visual>
             <origin xyz="0 0 0" rpy="0 0 0"/>
@@ -84,8 +84,8 @@
         </inertial>
     </link>
-    <joint name="${tf_prefix}/camera_joint" type="fixed">
-        <origin xyz="${stand_length/2 - camera_width} 0 ${camera_height / 2.0}" rpy="0 ${camera_pitch} 0"/>
-        <parent link="${tf_prefix}/stand_link"/>
-        <child link="${tf_prefix}/camera_link"/>
+    <joint name="camera_joint" type="fixed">
+        <origin xyz="${body_length/2 - camera_width} 0 ${camera_height / 2.0}" rpy="0 ${camera_pitch} 0"/>
+        <parent link="body_link"/>
+        <child link="camera_link"/>
     </joint>
 </robot>

File: description/urdf/inertias.xacro (robot description, xacro)
@@ -19,3 +19,11 @@
         />
     </xacro:macro>
+    <!--Camera Inertia for the Box-->
+     <xacro:macro name="box_inertia" params="mass length width height">
+        <inertia
+            ixx="${mass * (height*height + length*length)/12.0}" ixy="0.0" ixz="0.0"
+            iyx="0.0" iyy="${mass * (width*width + length*length)/12.0}" iyz="0.0"
+            izx="0.0" izy="0.0" izz="${mass * (width*width + height*height)/12.0}"
+        />
+    </xacro:macro>
 </robot>

File: description/urdf/plugins.gazebo.xacro (robot description, xacro)
@@ -95,5 +95,5 @@
                 <depthImageInfoTopicName>${depth_info_topicName}</depthImageInfoTopicName>
                 <pointCloudTopicName>${depth_points_topicName}</pointCloudTopicName>
-                <frameName>${tf_prefix}/${frameName}</frameName>
+                <frameName>photon/camera_link</frameName>
                 <hackBaseline>${camera_length}</hackBaseline>
                 <!-- TODO: Get distortion parameters from real camera -->

Commit message: applied new plugin

File: description/urdf/constants.xacro (robot description, xacro)
@@ -8,9 +8,15 @@
     <xacro:property name="wheel_radius" value="0.0635"/>
     <xacro:property name="thickness" value="0.1016"/>
+    <!-- Axle Positions -->
+    <xacro:property name="axel_offset" value="0.05"/>
+    <xacro:property name="steer_offset" value="0.02"/>
     <!-- Steer dimensions -->
-    <xacro:property name="steer_radius" value="0.05" />
-    <xacro:property name="steer_thickness" value="0.02" />
+    <xacro:property name="steer_radius" value="0.05"/>
+    <xacro:property name="steer_thickness" value="0.02"/>
+    <xacro:property name="steer_mass" value="1"/>
+    <!-- Steer properties -->
+    <xacro:property name="steer_velocity" value="5.0"/>
     <xacro:property name="steer_effort"   value="10.0"/>
-    <xacro:property name="steer_velocity" value="5.0"/>
+    <xacro:property name="steer_limit_deg"   value="90.0"/>
     <xacro:property name="deg_to_rad" value="0.01745329251994329577"/>
 </robot>

File: description/urdf/photon.urdf.xacro (robot description, xacro)
@@ -1,4 +1,4 @@
 <?xml version="1.0"?>
-<robot name="robot" xmlns:xacro="http://www.ros.org/wiki/xacro">
+<robot name="photon" xmlns:xacro="http://www.ros.org/wiki/xacro">
 <!--
 Robot model taken from http://wiki.ros.org/pr2_mechanism/Tutorials/SImple%20URDF-Controller%20Example
@@ -10,7 +10,4 @@
     <xacro:include filename="$(find description)/urdf/plugins.gazebo.xacro"/>
     <xacro:property name="deg_to_rad" value="0.01745329251994329577"/>
-    <!-- Constants for robot dimensions -->
-    <xacro:property name="axel_offset" value="0.05" /> <!-- Space btw top of beam and the each joint -->
-    <xacro:property name="steer_offset" value="0.02" /> <!-- Link 1 -->
     <!-- Links: inertial,visual,collision -->
     <link name="base_link">
@@ -42,8 +39,10 @@
     <xacro:front_wheel_lr name="front_left" parent="base" length="${fb_separation}"
         width="${lr_separation}" right_left="-1" steer_height="${wheel_radius+steer_offset}"/>
-    <xacro:rear_wheel_lr name="rear_right" parent="base" length="${fb_separation}"
-        width="${lr_separation}" right_left="1"/>
-    <xacro:rear_wheel_lr name="rear_left" parent="base" length="${fb_separation}"
-        width="${lr_separation}" right_left="-1"/>
+    <xacro:rear_wheel_lr name="rear_right" parent="base">
+        <origin xyz="${-fb_separation/2} ${lr_separation/2} ${height_to_wheel}" rpy="0 0 0"/>
+    </xacro:rear_wheel_lr>
+    <xacro:rear_wheel_lr name="rear_left" parent="base">
+        <origin xyz="${-fb_separation/2} ${-1*(lr_separation/2)} ${height_to_wheel}" rpy="0 0 0"/>
+    </xacro:rear_wheel_lr>
     <!-- Colour -->
     <gazebo reference="base_link">

File: description/urdf/photon_wheels.urdf.xacro (robot description, xacro)
@@ -1,4 +1,4 @@
 <?xml version="1.0"?>
-<robot xmlns:xacro="http://www.ros.org/wiki/xacro">
+<robot name="wheel" xmlns:xacro="http://www.ros.org/wiki/xacro">
   <!-- Includes -->
   <xacro:include filename="$(find description)/urdf/constants.xacro"/>
@@ -7,21 +7,23 @@
   <xacro:macro name="front_steer" params="name parent length steer_height">
     <link name="${name}_steer_link">
-      <inertial>
-        <origin xyz="0 0 0" rpy="0 0 0"/>
-        <mass value="1"/>
-        <inertia ixx="0.2" ixy="0" ixz="0" iyy="0.2" iyz="0" izz="0.2"/>
-      </inertial>
-      <visual>
-        <origin xyz="0 0 0" rpy="0 0 0"/>
-        <geometry>
-          <cylinder radius="${steer_radius}" length="${steer_thickness}"/>
-        </geometry>
-      </visual>
-      <collision>
-        <origin xyz="0 0 0" rpy="0 0 0"/>
-        <geometry>
-          <cylinder radius="${steer_radius}" length="${steer_thickness}"/>
-        </geometry>
-      </collision>
+      <visual>
+        <origin xyz="0 0 0" rpy="0 0 0"/>
+        <geometry>
+          <cylinder radius="${steer_radius}" length="${steer_thickness}"/>
+        </geometry>
+      </visual>
+      <collision>
+        <origin xyz="0 0 0" rpy="0 0 0"/>
+        <geometry>
+          <cylinder radius="${steer_radius}" length="${steer_thickness}"/>
+        </geometry>
+      </collision>
+      <inertial>
+        <origin xyz="0 0 0" rpy="0 0 0"/>
+        <mass value="${steer_mass}"/>
+        <inertia ixx="${steer_mass * (3.0 * steer_radius * steer_radius + steer_thickness * steer_thickness) / 12.0}"                 ixy="0" ixz="0"
+                iyy="${steer_mass * (3.0 * steer_radius * steer_radius + steer_thickness * steer_thickness) / 12.0}" iyz="0"
+                izz="${steer_mass * (steer_radius * steer_radius) / 2.0}"/>
+      </inertial>
     </link>
     <joint name="${name}_steer_joint" type="revolute">
@@ -34,4 +36,14 @@
              velocity="${steer_velocity}"/>
     </joint>
+    <transmission name="${name}_steer_joint_trans">
+      <type>transmission_interface/SimpleTransmission</type>
+      <actuator name="${name}_steer_joint_motor">
+        <mechanicalReduction>1</mechanicalReduction>
+        <hardwareInterface>hardware_interface/PositionJointInterface</hardwareInterface>
+      </actuator>
+      <joint name="${name}_steer_joint">
+        <hardwareInterface>hardware_interface/PositionJointInterface</hardwareInterface>
+      </joint>
+    </transmission>
     <gazebo reference="${name}_steer_link">
       <material>Gazebo/Yellow</material>
@@ -41,21 +53,23 @@
   <xacro:macro name="front_wheel_lr" params="name parent length width right_left steer_height">
     <link name="${name}_steer_link">
-      <inertial>
-        <origin xyz="0 0 0" rpy="0 0 0"/>
-        <mass value="1"/>
-        <inertia ixx="0.2" ixy="0" ixz="0" iyy="0.2" iyz="0" izz="0.2"/>
-      </inertial>
-      <visual>
-        <origin xyz="0 0 0" rpy="0 0 0"/>
-        <geometry>
-          <cylinder radius="${steer_radius}" length="${steer_thickness}"/>
-        </geometry>
-      </visual>
-      <collision>
-        <origin xyz="0 0 0" rpy="0 0 0"/>
-        <geometry>
-          <cylinder radius="${steer_radius}" length="${steer_thickness}"/>
-        </geometry>
-      </collision>
+      <visual>
+        <origin xyz="0 0 0" rpy="0 0 0"/>
+        <geometry>
+          <cylinder radius="${steer_radius}" length="${steer_thickness}"/>
+        </geometry>
+      </visual>
+      <collision>
+        <origin xyz="0 0 0" rpy="0 0 0"/>
+        <geometry>
+          <cylinder radius="${steer_radius}" length="${steer_thickness}"/>
+        </geometry>
+      </collision>
+      <inertial>
+        <origin xyz="0 0 0" rpy="0 0 0"/>
+        <mass value="${steer_mass}"/>
+        <inertia ixx="${steer_mass * (3.0 * steer_radius * steer_radius + steer_thickness * steer_thickness) / 12.0}"                 ixy="0" ixz="0"
+                iyy="${steer_mass * (3.0 * steer_radius * steer_radius + steer_thickness * steer_thickness) / 12.0}" iyz="0"
+                izz="${steer_mass * (steer_radius * steer_radius) / 2.0}"/>
+      </inertial>
     </link>
     <joint name="${name}_steer_joint" type="revolute">
@@ -63,26 +77,25 @@
       <child link="${name}_steer_link"/>
       <origin xyz="${length/2} ${right_left*(width/2)} ${steer_height}" rpy="0 0 0"/>
-      <!--xacro:insert_block name="origin"/-->
       <axis xyz="0 0 1"/>
       <limit effort="${steer_effort}"
-             lower="${-180.0 * deg_to_rad}" upper="${180.0 * deg_to_rad}"
+             lower="${steer_limit_deg * deg_to_rad * -1.0}" upper="${steer_limit_deg * deg_to_rad}"
              velocity="${steer_velocity}"/>
     </joint>
     <link name="${name}_wheel_link">
+      <visual>
+        <origin xyz="0 0 0" rpy="0 0 0"/>
+        <geometry>
+          <mesh filename="package://description/urdf/meshes/Wheels.STL" scale="0.001 0.001 0.001"/>
+        </geometry>
+      </visual>
+      <collision>
+        <origin xyz="0 0 0" rpy="0 0 0"/>
+        <geometry>
+          <mesh filename="package://description/urdf/meshes/Wheels.STL" scale="0.001 0.001 0.001"/>
+        </geometry>
+      </collision>
       <inertial>
         <xacro:wheel_inertia/>
       </inertial>
-      <visual>
-        <origin xyz="0 0 0" rpy="0 0 0"/>
-        <geometry>
-          <mesh filename="package://description/urdf/meshes/Wheels.STL" scale="0.001 0.001 0.001"/>
-        </geometry>
-      </visual>
-      <collision>
-        <origin xyz="0 0 0" rpy="0 0 0"/>
-        <geometry>
-          <mesh filename="package://description/urdf/meshes/Wheels.STL" scale="0.001 0.001 0.001"/>
-        </geometry>
-      </collision>
     </link>
     <joint name="${name}_wheel_joint" type="continuous">
@@ -92,16 +105,24 @@
       <axis xyz="0 1 0"/>
     </joint>
-    <!-- Transmission is important to link the joints and the controller -->
-    <transmission name="${name}_steer_joint_trans" type="SimpleTransmission">
-      <actuator name="${name}_steer_joint_motor"/>
-      <joint name="${name}_steer_joint"/>
-      <mechanicalReduction>1</mechanicalReduction>
-      <motorTorqueConstant>1</motorTorqueConstant>
-    </transmission>
-    <transmission name="${name}_wheel_joint_trans" type="SimpleTransmission">
-      <actuator name="${name}_wheel_joint_motor"/>
-      <joint name="${name}_wheel_joint"/>
-      <mechanicalReduction>1</mechanicalReduction>
-      <motorTorqueConstant>1</motorTorqueConstant>
+    <!-- Transmissions -->
+    <transmission name="${name}_steer_joint_trans">
+      <type>transmission_interface/SimpleTransmission</type>
+      <actuator name="${name}_steer_joint_motor">
+        <mechanicalReduction>1</mechanicalReduction>
+        <hardwareInterface>hardware_interface/PositionJointInterface</hardwareInterface>
+      </actuator>
+      <joint name="${name}_steer_joint">
+        <hardwareInterface>hardware_interface/PositionJointInterface</hardwareInterface>
+      </joint>
+    </transmission>
+    <transmission name="${name}_wheel_joint_trans">
+      <type>transmission_interface/SimpleTransmission</type>
+      <actuator name="${name}_wheel_joint_motor">
+        <mechanicalReduction>1</mechanicalReduction>
+        <hardwareInterface>hardware_interface/VelocityJointInterface</hardwareInterface>
+      </actuator>
+      <joint name="${name}_wheel_joint">
+        <hardwareInterface>hardware_interface/VelocityJointInterface</hardwareInterface>
+      </joint>
     </transmission>
     <gazebo reference="${name}_steer_link">
@@ -115,19 +136,19 @@
   <xacro:macro name="rear_wheel" params="name parent *origin">
     <link name="${name}_wheel_link">
+      <visual>
+        <origin xyz="0 0 0" rpy="0 0 0"/>
+        <geometry>
+          <cylinder radius="${wheel_radius}" length="${thickness}"/>
+        </geometry>
+      </visual>
+      <collision>
+        <origin xyz="0 0 0" rpy="0 0 0"/>
+        <geometry>
+          <cylinder radius="${wheel_radius}" length="${thickness}"/>
+        </geometry>
+      </collision>
       <inertial>
         <xacro:wheel_inertia/>
       </inertial>
-      <visual>
-        <origin xyz="0 0 0" rpy="0 0 0"/>
-        <geometry>
-          <cylinder radius="${wheel_radius}" length="${thickness}"/>
-        </geometry>
-      </visual>
-      <collision>
-        <origin xyz="0 0 0" rpy="0 0 0"/>
-        <geometry>
-          <cylinder radius="${wheel_radius}" length="${thickness}"/>
-        </geometry>
-      </collision>
     </link>
     <joint name="${name}_wheel_joint" type="continuous">
@@ -137,10 +158,14 @@
       <axis xyz="0 0 1"/>
     </joint>
-    <!-- Transmission is important to link the joints and the controller -->
-    <transmission name="${name}_wheel_joint_trans" type="SimpleTransmission">
-      <actuator name="${name}_wheel_joint_motor"/>
-      <joint name="${name}_wheel_joint"/>
-      <mechanicalReduction>1</mechanicalReduction>
-      <motorTorqueConstant>1</motorTorqueConstant>
+    <!-- Transmission -->
+    <transmission name="${name}_wheel_joint_trans">
+      <type>transmission_interface/SimpleTransmission</type>
+      <actuator name="${name}_wheel_joint_motor">
+        <mechanicalReduction>1</mechanicalReduction>
+        <hardwareInterface>hardware_interface/VelocityJointInterface</hardwareInterface>
+      </actuator>
+      <joint name="${name}_wheel_joint">
+        <hardwareInterface>hardware_interface/VelocityJointInterface</hardwareInterface>
+      </joint>
     </transmission>
     <gazebo reference="${name}_wheel_link">
@@ -149,34 +174,38 @@
   </xacro:macro>
   <!-- Rear wheels -->
-  <xacro:macro name="rear_wheel_lr" params="name parent length width right_left">
+  <xacro:macro name="rear_wheel_lr" params="name parent *origin">
     <link name="${name}_wheel_link">
+      <visual>
+        <origin xyz="0 0 0" rpy="0 0 0"/>
+        <geometry>
+          <mesh filename="package://description/urdf/meshes/Wheels.STL" scale="0.001 0.001 0.001"/>
+        </geometry>
+      </visual>
+      <collision>
+        <origin xyz="0 0 0" rpy="0 0 0"/>
+        <geometry>
+          <mesh filename="package://description/urdf/meshes/Wheels.STL" scale="0.001 0.001 0.001"/>
+        </geometry>
+      </collision>
       <inertial>
         <xacro:wheel_inertia/>
       </inertial>
-      <visual>
-        <origin xyz="0 0 0" rpy="0 0 0"/>
-        <geometry>
-          <mesh filename="package://description/urdf/meshes/Wheels.STL" scale="0.001 0.001 0.001"/>
-        </geometry>
-      </visual>
-      <collision>
-        <origin xyz="0 0 0" rpy="0 0 0"/>
-        <geometry>
-          <mesh filename="package://description/urdf/meshes/Wheels.STL" scale="0.001 0.001 0.001"/>
-        </geometry>
-      </collision>
     </link>
     <joint name="${name}_wheel_joint" type="continuous">
       <parent link="${parent}_link"/>
       <child link="${name}_wheel_link"/>
-      <origin xyz="${-length/2} ${right_left*(width/2)} ${height_to_wheel}" rpy="0 0 0"/>
+      <xacro:insert_block name="origin"/>
       <axis xyz="0 1 0"/>
     </joint>
-    <!-- Transmission is important to link the joints and the controller -->
-    <transmission name="${name}_wheel_joint_trans" type="SimpleTransmission">
-      <actuator name="${name}_wheel_joint_motor"/>
-      <joint name="${name}_wheel_joint"/>
-      <mechanicalReduction>1</mechanicalReduction>
-      <motorTorqueConstant>1</motorTorqueConstant>
+    <!-- Transmission -->
+    <transmission name="${name}_wheel_joint_trans">
+      <type>transmission_interface/SimpleTransmission</type>
+      <actuator name="${name}_wheel_joint_motor">
+        <mechanicalReduction>1</mechanicalReduction>
+        <hardwareInterface>hardware_interface/VelocityJointInterface</hardwareInterface>
+      </actuator>
+      <joint name="${name}_wheel_joint">
+        <hardwareInterface>hardware_interface/VelocityJointInterface</hardwareInterface>
+      </joint>
     </transmission>
     <gazebo reference="${name}_wheel_link">

File: description/urdf/plugins.gazebo.xacro (robot description, xacro)
@@ -3,9 +3,12 @@
     <!-- Constants -->
     <xacro:include filename="$(find description)/urdf/constants.xacro"/>
-    <!-- Gazebo Controller -->
+    <!-- Ackermann steering controller -->
     <gazebo>
-        <plugin name="steer_bot_hardware_gazebo" filename="libgazebo_ros_control.so">
-            <robotNamespace>/</robotNamespace>
-            <robotSimType>steer_bot_hardware_gazebo/SteerBotHardwareGazebo</robotSimType>
+        <!-- Load ros_control plugin using the steer_bot_hardware_gazebo
+        implementation of the hardware_interface::RobotHW -->
+        <plugin name="gazebo_ros_control" filename="libgazebo_ros_control.so">
+        <robotNamespace>/</robotNamespace>
+        <robotSimType>steer_bot_hardware_gazebo/SteerBotHardwareGazebo</robotSimType>
+        <legacyModeNS>false</legacyModeNS>
         </plugin>
     </gazebo>
