Commit message: Corrected stereo camera to be in the correct location and with the correct set up

File: description/urdf/constants.xacro (robot description, xacro)
@@ -21,4 +21,5 @@
     <xacro:property name="laser_min_range" value="0.06"/>
     <xacro:property name="laser_max_range" value="4.095"/>
+    <!-- STEREO CAMERA -->
     <xacro:property name="camera_mass" value="0.1587573"/>
     <xacro:property name="camera_length" value="0.175"/>
@@ -26,19 +27,18 @@
     <xacro:property name="camera_height" value="0.033"/>
     <xacro:property name="camera_pitch" value="${15 * pi/180}"/>
-    <!-- CAMERA PLUG - IN-->
-    <xacro:property name="image_refresh" value="60"/>
+    <xacro:property name="camera_update_rate" value="60"/>
+    <xacro:property name="camera_hfov" value="${90 * pi/180}"/>
+    <xacro:property name="stereo_offset" value="${camera_length / 2.0}"/>    <!-- Distance between left and right cameras -->
     <xacro:property name="image_width" value="3840"/>
     <xacro:property name="image_height" value="1080"/>
     <xacro:property name="image_format" value="R8G8B8"/>
-    <xacro:property name="image_hfov" value="${90 * pi/180}"/>
-    <xacro:property name="name" value="camera/camera_node"/>
+    <xacro:property name="camera_ns" value="camera/camera_node"/>
     <xacro:property name="always_on" value="true"/>
-    <xacro:property name="update_rate" value="0"/>
     <xacro:property name="image_topicName" value="image_raw_color"/>
     <xacro:property name="image_info_topicName" value="camera_info"/>
     <xacro:property name="depth_topicName" value="depth/image_raw"/>
     <xacro:property name="depth_info_topicName" value="depth/camera_info"/>
-    <xacro:property name="depth_points_topicName" value="depth/points"/>
-    <xacro:property name="frameName" value="zed_camera_link_optical"/>
+    <xacro:property name="pointcloud_topicName" value="pointcloud"/>
+    <xacro:property name="camera_left_optical_frame" value="camera_left_link_optical"/>
     <!-- IMU -->
     <xacro:property name="imu_update_rate" value="128"/>

File: description/urdf/inertias.xacro (robot description, xacro)
@@ -19,10 +19,11 @@
         />
     </xacro:macro>
-    <!--Camera Inertia for the Box-->
-     <xacro:macro name="box_inertia" params="mass length width height">
+    <!--Box Shaped Objects -->
+    <xacro:macro name="box_inertia" params="mass length width height">
+        <mass value="${mass}"/>
         <inertia
-            ixx="${mass * (height*height + length*length)/12.0}" ixy="0.0" ixz="0.0"
-            iyx="0.0" iyy="${mass * (width*width + length*length)/12.0}" iyz="0.0"
-            izx="0.0" izy="0.0" izz="${mass * (width*width + height*height)/12.0}"
+            ixx="${mass * (height*height + length*length) / 12.0}" ixy="0.0" ixz="0.0"
+            iyy="${mass * (width*width + length*length) / 12.0}" iyz="0.0"
+            izz="${mass * (width*width + height*height) / 12.0}"
         />
     </xacro:macro>

File: description/urdf/photon.urdf.xacro (robot description, xacro)
@@ -4,4 +4,5 @@
     <xacro:include filename="$(find description)/urdf/constants.xacro"/>
     <xacro:include filename="$(find description)/urdf/inertias.xacro"/>
+    <xacro:include filename="$(find description)/urdf/materials.xacro"/>
     <xacro:include filename="$(find description)/urdf/plugins.gazebo.xacro"/>
     <link name="base_link"/>
@@ -31,5 +32,5 @@
     <!-- Wheels -->
     <xacro:include filename="$(find description)/urdf/wheels.urdf.xacro"/>
-     <!-- LIDAR -->
+    <!-- LIDAR -->
     <link name="lidar_link">
         <visual>
@@ -38,6 +39,6 @@
                 <box size="0.03 0.03 0.03" />
             </geometry>
-            <material name="Cyan">
-                <color rgba="0 1.0 1.0 1.0"/>
+            <material name="Grey">
+                <color rgba="0.75 0.75 0.75 1.0"/>
             </material>
         </visual>
@@ -48,5 +49,5 @@
         <origin xyz="${fb_separation/2} 0 ${-height_to_wheel/2}" rpy="0 0 0"/>
     </joint>
-     <!-- IMU -->
+    <!-- IMU -->
     <link name="imu_link">
         <visual>
@@ -55,6 +56,6 @@
                 <box size="0.03 0.03 0.03" />
             </geometry>
-            <material name="Cyan">
-                <color rgba="0 0.0 1.0 1.0"/>
+            <material name="Green">
+                <color rgba="0.0 1.0 0.0 1.0"/>
             </material>
         </visual>
@@ -65,11 +66,15 @@
         <origin xyz="0 0 ${-height_to_wheel}" rpy="0 0 0"/>
     </joint>
-    <!-- ZED Camera -->
+    <!-- STEREO CAMERA -->
+    <!-- NOTE: this frame is for convenience, multicamera will use the subsequent left camera frames -->
     <link name="camera_link">
         <visual>
             <origin xyz="0 0 0" rpy="0 0 0"/>
             <geometry>
-            <box size="${camera_width} ${camera_length} ${camera_height}"/>
+                <box size="${camera_width} ${camera_length} ${camera_height}"/>
             </geometry>
+            <material name="Blue">
+                <color rgba="0.0 0.0 1.0 1.0"/>
+            </material>
         </visual>
         <collision>
@@ -81,11 +86,25 @@
         <inertial>
             <xacro:box_inertia mass="${camera_mass}" length="${camera_length}" width="${camera_width}" height="${camera_height}"/>
-            <mass value="${camera_mass}"/>
         </inertial>
     </link>
     <joint name="camera_joint" type="fixed">
-        <origin xyz="${body_length/2 - camera_width} 0 ${camera_height / 2.0}" rpy="0 ${camera_pitch} 0"/>
         <parent link="body_link"/>
         <child link="camera_link"/>
+        <origin xyz="${body_length / 2.0 - camera_width} 0 ${-height_to_wheel + camera_height / 2.0}" rpy="0 ${camera_pitch} 0"/>
+    </joint>
+    <!-- Generate Left Camera frame -->
+    <!-- NOTE: specify frame of left camera because right one is specified relative to it by the multicamera plugin -->
+    <link name="camera_left_link"/>
+    <joint name="camera_left_link_joint" type="fixed">
+        <parent link="camera_link"/>
+        <child link="camera_left_link"/>
+        <origin xyz="0 ${stereo_offset / 2.0} 0" rpy="0 0 0"/>
+    </joint>
+    <!-- Generate the Optical frame http://www.ros.org/reps/rep-0103.html#suffix-frames so that ros and opencv can operate on the camera frame correctly -->
+    <link name="camera_left_link_optical"/>
+    <joint name="camera_left_link_optical_joint" type="fixed">
+        <parent link="camera_left_link"/>
+        <child link="camera_left_link_optical"/>
+        <origin xyz="0 0 0" rpy="${-pi/2} 0 ${-pi/2}"/>
     </joint>
 </robot>

File: description/urdf/plugins.gazebo.xacro (robot description, xacro)
@@ -45,6 +45,6 @@
             <plugin filename="libgazebo_ros_imu_sensor.so" name="imu_plugin">
                 <topicName>imu/data</topicName>
-                <bodyName>photon/imu_link</bodyName>
-                <frameName>photon/imu_link</frameName>
+                <bodyName>imu_link</bodyName>
+                <frameName>imu_link</frameName>
                 <updateRateHZ>${imu_update_rate}</updateRateHZ>
                 <gaussianNoise>0.0</gaussianNoise>
@@ -56,45 +56,48 @@
         </sensor>
     </gazebo>
-<!--Stereo Camera-->
-    <!-- Gazebo multicamera plugin -->
-    <gazebo reference="camera_link">
+    <!--Stereo Camera-->
+    <!-- NOTE:
+    it is assumed that the left camera is at the origin specified by "frameName" (or
+    referenced by gazebo) and that the right camera is "hackBaseline" away from it
+    -->
+    <gazebo reference="camera_left_link">
         <sensor type="multicamera" name="stereo_camera">
-            <update_rate>${image_refresh}</update_rate>
+            <update_rate>${camera_update_rate}</update_rate>
             <camera name="left">
-            <horizontal_fov>${image_hfov}</horizontal_fov>
-            <image>
-                <width>${image_width}</width>
-                <height>${image_height}</height>
-                <format>${image_format}</format>
-            </image>
-            <clip>
-                <near>0.02</near>
-                <far>300</far>
-            </clip>
+                <horizontal_fov>${camera_hfov}</horizontal_fov>
+                <image>
+                    <width>${image_width}</width>
+                    <height>${image_height}</height>
+                    <format>${image_format}</format>
+                </image>
+                <clip>
+                    <near>0.02</near>
+                    <far>300</far>
+                </clip>
             </camera>
             <camera name="right">
-            <pose>0 ${-camera_length} 0 0 0 0</pose>
-            <horizontal_fov>${image_hfov}</horizontal_fov>
-            <image>
-                <width>${image_width}</width>
-                <height>${image_height}</height>
-                <format>${image_format}</format>
-            </image>
-            <clip>
-                <near>0.02</near>
-                <far>300</far>
-            </clip>
+                <pose>0 -${stereo_offset} 0 0 0 0</pose>
+                <horizontal_fov>${camera_hfov}</horizontal_fov>
+                <image>
+                    <width>${image_width}</width>
+                    <height>${image_height}</height>
+                    <format>${image_format}</format>
+                </image>
+                <clip>
+                    <near>0.02</near>
+                    <far>300</far>
+                </clip>
             </camera>
             <plugin name="stereo_camera_controller" filename="libgazebo_ros_multicamera.so">
-                <cameraName>${name}</cameraName>
+                <cameraName>${camera_ns}</cameraName>
                 <alwaysOn>${always_on}</alwaysOn>
-                <updateRate>${update_rate}</updateRate>
+                <updateRate>${camera_update_rate}</updateRate>
                 <imageTopicName>${image_topicName}</imageTopicName>
                 <cameraInfoTopicName>${image_info_topicName}</cameraInfoTopicName>
                 <depthImageTopicName>${depth_topicName}</depthImageTopicName>
                 <depthImageInfoTopicName>${depth_info_topicName}</depthImageInfoTopicName>
-                <pointCloudTopicName>${depth_points_topicName}</pointCloudTopicName>
-                <frameName>camera_link</frameName>
-                <hackBaseline>${camera_length}</hackBaseline>
+                <pointCloudTopicName>${pointcloud_topicName}</pointCloudTopicName>
+                <frameName>${camera_left_optical_frame}</frameName>
+                <hackBaseline>${stereo_offset}</hackBaseline>
                 <!-- TODO: Get distortion parameters from real camera -->
                 <distortionK1>0.0</distortionK1>

Commit message: Code cleanup

File: description/urdf/constants.xacro (robot description, xacro)
@@ -26,12 +26,12 @@
     <xacro:property name="camera_width" value="0.03"/>
     <xacro:property name="camera_height" value="0.033"/>
-    <xacro:property name="camera_pitch" value="${15 * pi/180}"/>
-    <xacro:property name="camera_update_rate" value="60"/>
+    <xacro:property name="camera_pitch" value="${5 * pi/180}"/>
+    <xacro:property name="camera_update_rate" value="30"/>
     <xacro:property name="camera_hfov" value="${90 * pi/180}"/>
     <xacro:property name="stereo_offset" value="${camera_length / 2.0}"/>    <!-- Distance between left and right cameras -->
-    <xacro:property name="image_width" value="3840"/>
+    <xacro:property name="image_width" value="1920"/>
     <xacro:property name="image_height" value="1080"/>
     <xacro:property name="image_format" value="R8G8B8"/>
-    <xacro:property name="camera_ns" value="camera/camera_node"/>
+    <xacro:property name="camera_ns" value="camera/camera_node"/>  <!-- Use a name representative of the camera being used -->
     <xacro:property name="always_on" value="true"/>
     <xacro:property name="image_topicName" value="image_raw_color"/>

Commit message: PHN5 - RGBD Camera (#15)
* checking branch

* added launch and rviz files for rgbd camera

* all files are in. code based on caffeine ZED camera. error when launching

* fixed some errors

* push routine

* changes allows for launching camera not there

* Spawns in RVIZ, need to change settings, look into how gazebo spawns it. Error that appears is benign

* Corrected stereo camera to be in the correct location and with the correct set up

* Code cleanup

Co-authored-by: Paula Santas Rodriguez <psantasr>
Co-authored-by: Marie Joy Cuevas <cuevas.mariejoy@gmail.com>
Co-authored-by: Erick Mejia Uzeda <erickmu1@hotmail.com>

File: description/urdf/constants.xacro (robot description, xacro)
@@ -21,4 +21,24 @@
     <xacro:property name="laser_min_range" value="0.06"/>
     <xacro:property name="laser_max_range" value="4.095"/>
+    <!-- STEREO CAMERA -->
+    <xacro:property name="camera_mass" value="0.1587573"/>
+    <xacro:property name="camera_length" value="0.175"/>
+    <xacro:property name="camera_width" value="0.03"/>
+    <xacro:property name="camera_height" value="0.033"/>
+    <xacro:property name="camera_pitch" value="${5 * pi/180}"/>
+    <xacro:property name="camera_update_rate" value="30"/>
+    <xacro:property name="camera_hfov" value="${90 * pi/180}"/>
+    <xacro:property name="stereo_offset" value="${camera_length / 2.0}"/>    <!-- Distance between left and right cameras -->
+    <xacro:property name="image_width" value="1920"/>
+    <xacro:property name="image_height" value="1080"/>
+    <xacro:property name="image_format" value="R8G8B8"/>
+    <xacro:property name="camera_ns" value="camera/camera_node"/>  <!-- Use a name representative of the camera being used -->
+    <xacro:property name="always_on" value="true"/>
+    <xacro:property name="image_topicName" value="image_raw_color"/>
+    <xacro:property name="image_info_topicName" value="camera_info"/>
+    <xacro:property name="depth_topicName" value="depth/image_raw"/>
+    <xacro:property name="depth_info_topicName" value="depth/camera_info"/>
+    <xacro:property name="pointcloud_topicName" value="pointcloud"/>
+    <xacro:property name="camera_left_optical_frame" value="camera_left_link_optical"/>
     <!-- IMU -->
     <xacro:property name="imu_update_rate" value="128"/>

File: description/urdf/inertias.xacro (robot description, xacro)
@@ -19,3 +19,12 @@
         />
     </xacro:macro>
+    <!--Box Shaped Objects -->
+    <xacro:macro name="box_inertia" params="mass length width height">
+        <mass value="${mass}"/>
+        <inertia
+            ixx="${mass * (height*height + length*length) / 12.0}" ixy="0.0" ixz="0.0"
+            iyy="${mass * (width*width + length*length) / 12.0}" iyz="0.0"
+            izz="${mass * (width*width + height*height) / 12.0}"
+        />
+    </xacro:macro>
 </robot>

File: description/urdf/plugins.gazebo.xacro (robot description, xacro)
@@ -45,6 +45,6 @@
             <plugin filename="libgazebo_ros_imu_sensor.so" name="imu_plugin">
                 <topicName>imu/data</topicName>
-                <bodyName>photon/imu_link</bodyName>
-                <frameName>photon/imu_link</frameName>
+                <bodyName>imu_link</bodyName>
+                <frameName>imu_link</frameName>
                 <updateRateHZ>${imu_update_rate}</updateRateHZ>
                 <gaussianNoise>0.0</gaussianNoise>
@@ -56,3 +56,56 @@
         </sensor>
     </gazebo>
+    <!--Stereo Camera-->
+    <!-- NOTE:
+    it is assumed that the left camera is at the origin specified by "frameName" (or
+    referenced by gazebo) and that the right camera is "hackBaseline" away from it
+    -->
+    <gazebo reference="camera_left_link">
+        <sensor type="multicamera" name="stereo_camera">
+            <update_rate>${camera_update_rate}</update_rate>
+            <camera name="left">
+                <horizontal_fov>${camera_hfov}</horizontal_fov>
+                <image>
+                    <width>${image_width}</width>
+                    <height>${image_height}</height>
+                    <format>${image_format}</format>
+                </image>
+                <clip>
+                    <near>0.02</near>
+                    <far>300</far>
+                </clip>
+            </camera>
+            <camera name="right">
+                <pose>0 -${stereo_offset} 0 0 0 0</pose>
+                <horizontal_fov>${camera_hfov}</horizontal_fov>
+                <image>
+                    <width>${image_width}</width>
+                    <height>${image_height}</height>
+                    <format>${image_format}</format>
+                </image>
+                <clip>
+                    <near>0.02</near>
+                    <far>300</far>
+                </clip>
+            </camera>
+            <plugin name="stereo_camera_controller" filename="libgazebo_ros_multicamera.so">
+                <cameraName>${camera_ns}</cameraName>
+                <alwaysOn>${always_on}</alwaysOn>
+                <updateRate>${camera_update_rate}</updateRate>
+                <imageTopicName>${image_topicName}</imageTopicName>
+                <cameraInfoTopicName>${image_info_topicName}</cameraInfoTopicName>
+                <depthImageTopicName>${depth_topicName}</depthImageTopicName>
+                <depthImageInfoTopicName>${depth_info_topicName}</depthImageInfoTopicName>
+                <pointCloudTopicName>${pointcloud_topicName}</pointCloudTopicName>
+                <frameName>${camera_left_optical_frame}</frameName>
+                <hackBaseline>${stereo_offset}</hackBaseline>
+                <!-- TODO: Get distortion parameters from real camera -->
+                <distortionK1>0.0</distortionK1>
+                <distortionK2>0.0</distortionK2>
+                <distortionK3>0.0</distortionK3>
+                <distortionT1>0.0</distortionT1>
+                <distortionT2>0.0</distortionT2>
+            </plugin>
+        </sensor>
+    </gazebo>
 </robot>
