Commit message: PHN4 - Simulate Motor + Drive (#13)
* added diff_drive_controller and rqt_steering

* diff_drive controller working

* changed to front wheels and file name

* added rviz view in simulate.launch file

* edited naming

* added ackermann steering controller and corresponding urdf and launch files

* gazebo cylinder for rear wheel link instead of mesh

* fixed rviz

* Updated readme

* updated rviz, removed unused files

* updated rviz and removed unused files

* added plugin

* added ackerman steering repo as linked by Jimin. The test files work, hasn't been imported over to our own simulate files yet

* applied new plugin

* edited cloning instructions

* added rviz view to launch file

* added steer drive ros

* edited format

* minor edits

* new lines

* Removed a recurring INFO print statement from steer_drive_ros

* Restructured how ackermann steering was integrated. Note that moving Photon is rather unstable

Co-authored-by: EsteBran <32085355+EsteBran@users.noreply.github.com>
Co-authored-by: EsteBran <tawseefhanif@gmail.com>
Co-authored-by: Erick Mejia Uzeda <erickmu1@hotmail.com>

File: description/urdf/constants.xacro (robot description, xacro)
@@ -15,4 +15,18 @@
     <xacro:property name="lr_separation" value="0.304"/>
     <xacro:property name="height_to_wheel" value="-0.1135"/>
+    <!-- Wheel dimensions -->
+    <xacro:property name="wheel_radius" value="0.0635"/>
+    <xacro:property name="thickness" value="0.1016"/>
+    <!-- Axle Positions: Check with Mech Team, currently made up -->
+    <xacro:property name="axel_offset" value="0.05"/>
+    <xacro:property name="steer_offset" value="0.02"/>
+    <!-- Steer dimensions: Check with Mech Team, currently made up -->
+    <xacro:property name="steer_radius" value="0.05"/>
+    <xacro:property name="steer_thickness" value="0.02"/>
+    <xacro:property name="steer_mass" value="1.0"/>
+    <!-- Steer properties: Check with Mech Team, currently made up -->
+    <xacro:property name="steer_velocity" value="5.0"/>
+    <xacro:property name="steer_effort" value="10.0"/>
+    <xacro:property name="steer_limit" value="${90.0 * pi/180}"/>
     <!-- LIDAR -->
     <xacro:property name="laser_visualize" value="false"/>

File: description/urdf/inertias.xacro (robot description, xacro)
@@ -28,3 +28,12 @@
         />
     </xacro:macro>
+    <!-- Cylinder Shaped Objects -->
+    <xacro:macro name="cylinder_inertia" params="mass radius length">
+        <mass value="${mass}"/>
+        <inertia
+            ixx="${mass * (3.0 * radius*radius + length*length) / 12.0}" ixy="0.0" ixz="0.0"
+            iyy="${mass * (3.0 * radius*radius + length*length) / 12.0}" iyz="0.0"
+            izz="${mass * radius*radius / 2.0}"
+        />
+    </xacro:macro>
 </robot>

File: description/urdf/materials.xacro (robot description, xacro)
@@ -1,4 +1,17 @@
 <?xml version="1.0"?>
 <robot name="materials" xmlns:xacro="http://ros.org/wiki/xacro">
+    <!-- Ackermann Steering -->
+    <gazebo reference="front_steer_link">
+        <material>Gazebo/Yellow</material>
+    </gazebo>
+    <gazebo reference="front_left_steer_link">
+        <material>Gazebo/Yellow</material>
+    </gazebo>
+    <gazebo reference="front_right_steer_link">
+        <material>Gazebo/Yellow</material>
+    </gazebo>
+    <gazebo reference="virtual_rear_wheel_link">
+        <material>Gazebo/Yellow</material>
+    </gazebo>
     <!-- LIDAR -->
     <gazebo reference="lidar_link">

File: description/urdf/photon.urdf.xacro (robot description, xacro)
@@ -1,4 +1,4 @@
 <?xml version="1.0"?>
-<robot name="cybertruck" xmlns:xacro="http://ros.org/wiki/xacro">
+<robot name="photon" xmlns:xacro="http://ros.org/wiki/xacro">
     <!-- Includes -->
     <xacro:include filename="$(find description)/urdf/constants.xacro"/>
@@ -12,5 +12,5 @@
             <origin xyz="0 0 0" rpy="0 0 0"/>
             <geometry>
-                <mesh filename="package://description/urdf/meshes/StampedeBody.stl" scale="0.001 0.001 0.001"/>
+                <mesh filename="package://description/urdf/meshes/Body.STL" scale="0.001 0.001 0.001"/>
             </geometry>
         </visual>
@@ -18,5 +18,5 @@
             <origin xyz="0 0 0" rpy="0 0 0"/>
             <geometry>
-                <mesh filename="package://description/urdf/meshes/StampedeBody.stl" scale="0.001 0.001 0.001"/>
+                <mesh filename="package://description/urdf/meshes/Body.STL" scale="0.001 0.001 0.001"/>
             </geometry>
         </collision>

File: description/urdf/plugins.gazebo.xacro (robot description, xacro)
@@ -3,4 +3,13 @@
     <!-- Constants -->
     <xacro:include filename="$(find description)/urdf/constants.xacro"/>
+    <!-- Ackermann Steering Controller -->
+    <gazebo>
+        <!-- Load ros_control plugin using the steer_bot_hardware_gazebo implementation of the hardware_interface::RobotHW -->
+        <plugin name="gazebo_ros_control" filename="libgazebo_ros_control.so">
+            <robotNamespace>/</robotNamespace>
+            <robotSimType>steer_bot_hardware_gazebo/SteerBotHardwareGazebo</robotSimType>
+            <legacyModeNS>false</legacyModeNS>
+        </plugin>
+    </gazebo>
     <!-- LIDAR -->
     <gazebo reference="lidar_link">

File: description/urdf/wheels.urdf.xacro (robot description, xacro)
@@ -1,9 +1,55 @@
 <?xml version="1.0"?>
-<robot name="cybertruck_wheels" xmlns:xacro="http://ros.org/wiki/xacro">
+<robot name="wheels" xmlns:xacro="http://ros.org/wiki/xacro">
     <!-- Includes -->
     <xacro:include filename="$(find description)/urdf/constants.xacro"/>
     <xacro:include filename="$(find description)/urdf/inertias.xacro"/>
+    <!-- TODO: see if virtual objects can be invisible and have small masses (as to not affect Photon in anyway other than enable ackermann steering) -->
+    <!-- MACRO -->
+    <xacro:property name="steer_height" value="${wheel_radius + steer_offset}"/>
+    <!-- Steer macro -->
+    <xacro:macro name="Steer" params="name steer_limit *origin">
+        <!-- Steer link -->
+        <link name="${name}_steer_link">
+            <visual>
+                <origin xyz="0 0 0" rpy="0 0 0"/>
+                <geometry>
+                    <cylinder radius="${steer_radius}" length="${steer_thickness}"/>
+                </geometry>
+                <material name="Yellow">
+                    <color rgba="1.0 1.0 0.0 1.0"/>
+                </material>
+            </visual>
+            <collision>
+                <origin xyz="0 0 0" rpy="0 0 0"/>
+                <geometry>
+                    <cylinder radius="${steer_radius}" length="${steer_thickness}"/>
+                </geometry>
+            </collision>
+            <inertial>
+                <xacro:cylinder_inertia mass="${steer_mass}" radius="${steer_radius}" length="${steer_thickness}"/>
+            </inertial>
+        </link>
+        <!-- Steer joint -->
+        <joint name="${name}_steer_joint" type="revolute">
+            <parent link="body_link"/>
+            <child link="${name}_steer_link"/>
+            <xacro:insert_block name="origin"/>
+            <axis xyz="0 0 1"/>
+            <limit effort="${steer_effort}" lower="-${steer_limit}" upper="${steer_limit}" velocity="${steer_velocity}"/>
+        </joint>
+        <!-- Transmission -->
+        <transmission name="${name}_steer_joint_trans">
+            <type>transmission_interface/SimpleTransmission</type>
+            <actuator name="${name}_steer_joint_motor">
+                <mechanicalReduction>1</mechanicalReduction>
+                <hardwareInterface>hardware_interface/PositionJointInterface</hardwareInterface>
+            </actuator>
+            <joint name="${name}_steer_joint">
+                <hardwareInterface>hardware_interface/PositionJointInterface</hardwareInterface>
+            </joint>
+        </transmission>
+    </xacro:macro>
     <!-- Wheel macro -->
-    <xacro:macro name="Wheel" params="fb lr">
+    <xacro:macro name="Wheel" params="fb lr *parent *origin">
         <!-- Wheel link -->
         <link name="${fb}_${lr}_wheel_link">
@@ -11,5 +57,5 @@
                 <origin xyz="0 0 0" rpy="0 0 0"/>
                 <geometry>
-                    <mesh filename="package://description/urdf/meshes/Wheel.stl" scale="0.001 0.001 0.001"/>
+                    <mesh filename="package://description/urdf/meshes/Wheels.STL" scale="0.001 0.001 0.001"/>
                 </geometry>
             </visual>
@@ -17,5 +63,5 @@
                 <origin xyz="0 0 0" rpy="0 0 0"/>
                 <geometry>
-                    <mesh filename="package://description/urdf/meshes/Wheel.stl" scale="0.001 0.001 0.001"/>
+                    <mesh filename="package://description/urdf/meshes/Wheels.STL" scale="0.001 0.001 0.001"/>
                 </geometry>
             </collision>
@@ -26,16 +72,85 @@
         <!-- Wheel joint -->
         <joint name="${fb}_${lr}_wheel_joint" type="continuous">
-            <parent link="body_link"/>
+            <xacro:insert_block name="parent"/>
             <child link="${fb}_${lr}_wheel_link"/>
-            <origin xyz="${fb_separation/2 if fb == 'front' else -fb_separation/2}
-                    ${-lr_separation/2 if lr == 'left' else lr_separation/2}
-                    ${height_to_wheel}" rpy="0 0 0"/>
+            <xacro:insert_block name="origin"/>
             <axis xyz="0 1 0"/>
         </joint>
+        <!-- Transmission -->
+        <transmission name="${fb}_${lr}_wheel_joint_trans">
+            <type>transmission_interface/SimpleTransmission</type>
+            <actuator name="${fb}_${lr}_wheel_joint_motor">
+                <mechanicalReduction>1</mechanicalReduction>
+                <hardwareInterface>hardware_interface/VelocityJointInterface</hardwareInterface>
+            </actuator>
+            <joint name="${fb}_${lr}_wheel_joint">
+                <hardwareInterface>hardware_interface/VelocityJointInterface</hardwareInterface>
+            </joint>
+        </transmission>
     </xacro:macro>
-    <!-- Instantiate wheels -->
-    <xacro:Wheel fb="front" lr="left"/>
-    <xacro:Wheel fb="front" lr="right"/>
-    <xacro:Wheel fb="back" lr="left"/>
-    <xacro:Wheel fb="back" lr="right"/>
+    <!-- INSTANTIATION -->
+    <!-- Instantiate Front Steers (Ackermann Steering) -->
+    <xacro:Steer name="front" steer_limit="${180.0 * pi/180}">
+        <origin xyz="${fb_separation/2} 0 ${steer_height}" rpy="0 0 0"/>
+    </xacro:Steer>
+    <xacro:Steer name="front_left" steer_limit="${steer_limit}">
+        <origin xyz="${fb_separation/2} -${lr_separation/2} ${steer_height}" rpy="0 0 0"/>
+    </xacro:Steer>
+    <xacro:Steer name="front_right" steer_limit="${steer_limit}">
+        <origin xyz="${fb_separation/2} ${lr_separation/2} ${steer_height}" rpy="0 0 0"/>
+    </xacro:Steer>
+    <!-- Instantiate Virtual Rear Wheel (Ackermann Steering) -->
+    <link name="virtual_rear_wheel_link">
+        <visual>
+            <origin xyz="0 0 0" rpy="0 0 0"/>
+            <geometry>
+                <cylinder radius="${wheel_radius}" length="${thickness}"/>
+            </geometry>
+            <material name="Yellow">
+                <color rgba="1.0 1.0 0.0 1.0"/>
+            </material>
+        </visual>
+        <collision>
+            <origin xyz="0 0 0" rpy="0 0 0"/>
+            <geometry>
+                <cylinder radius="${wheel_radius}" length="${thickness}"/>
+            </geometry>
+        </collision>
+        <inertial>
+            <xacro:wheel_inertia/>
+        </inertial>
+    </link>
+    <joint name="virtual_rear_wheel_joint" type="continuous">
+        <parent link="body_link"/>
+        <child link="virtual_rear_wheel_link"/>
+        <origin xyz="-${fb_separation/2} 0 ${height_to_wheel}" rpy="${-90 * pi/180} 0 0"/>
+        <axis xyz="0 0 1"/>
+    </joint>
+    <transmission name="virtual_rear_wheel_joint_trans">
+        <type>transmission_interface/SimpleTransmission</type>
+        <actuator name="virtual_rear_wheel_joint_motor">
+            <mechanicalReduction>1</mechanicalReduction>
+            <hardwareInterface>hardware_interface/VelocityJointInterface</hardwareInterface>
+        </actuator>
+        <joint name="virtual_rear_wheel_joint">
+            <hardwareInterface>hardware_interface/VelocityJointInterface</hardwareInterface>
+        </joint>
+    </transmission>
+    <!-- Instantiate Physical Wheels -->
+    <xacro:Wheel fb="front" lr="left">
+        <parent link="front_left_steer_link"/>
+        <origin xyz="0 0 ${height_to_wheel - steer_height}" rpy="0 0 0"/>
+    </xacro:Wheel>
+    <xacro:Wheel fb="front" lr="right">
+        <parent link="front_right_steer_link"/>
+        <origin xyz="0 0 ${height_to_wheel - steer_height}" rpy="0 0 0"/>
+    </xacro:Wheel>
+    <xacro:Wheel fb="back" lr="left">
+        <parent link="body_link"/>
+        <origin xyz="-${fb_separation/2} -${lr_separation/2} ${height_to_wheel}" rpy="0 0 0"/>
+    </xacro:Wheel>
+    <xacro:Wheel fb="back" lr="right">
+        <parent link="body_link"/>
+        <origin xyz="-${fb_separation/2} ${lr_separation/2} ${height_to_wheel}" rpy="0 0 0"/>
+    </xacro:Wheel>
 </robot>
