Commit message: gazebo cylinder for rear wheel link instead of mesh

File: description/urdf/photon.urdf.xacro (robot description, xacro)
@@ -52,5 +52,5 @@
     steer_height="${wheel_radius+steer_offset}"/>
   <xacro:rear_wheel name="rear" parent="base">
-    <origin xyz="${-fb_separation/2} 0 0" rpy="0 0 0"/>
+    <origin xyz="${-fb_separation/2} 0 ${height_to_wheel}" rpy="${-90 * deg_to_rad} 0 0"/>
   </xacro:rear_wheel>
   <!-- Wheels -->

File: description/urdf/photon_wheels.urdf.xacro (robot description, xacro)
@@ -89,5 +89,5 @@
       <parent link="${name}_steer_link"/>
       <child link="${name}_wheel_link"/>
-      <origin xyz="0 0 ${-steer_height}" rpy="0 0 0"/>
+      <origin xyz="0 0 ${-steer_height+height_to_wheel}" rpy="0 0 0"/>
       <axis xyz="0 1 0"/>
     </joint>
@@ -121,5 +121,5 @@
         <origin xyz="0 0 0" rpy="0 0 0"/>
         <geometry>
-          <mesh filename="package://description/urdf/meshes/Wheelfxorigin.STL" scale="0.001 0.001 0.001"/>
+          <cylinder radius="${wheel_radius}" length="${thickness}"/>
         </geometry>
       </visual>
@@ -127,5 +127,5 @@
         <origin xyz="0 0 0" rpy="0 0 0"/>
         <geometry>
-          <mesh filename="package://description/urdf/meshes/Wheelfxorigin.STL" scale="0.001 0.001 0.001"/>
+          <cylinder radius="${wheel_radius}" length="${thickness}"/>
         </geometry>
       </collision>
@@ -135,5 +135,5 @@
       <child link="${name}_wheel_link"/>
       <xacro:insert_block name="origin"/>
-      <axis xyz="0 1 0"/>
+      <axis xyz="0 0 1"/>
     </joint>
     <!-- Transmission is important to link the joints and the controller -->
@@ -170,5 +170,5 @@
       <parent link="${parent}_link"/>
       <child link="${name}_wheel_link"/>
-      <origin xyz="${-length/2} ${right_left*(width/2)} 0" rpy="0 0 0"/>
+      <origin xyz="${-length/2} ${right_left*(width/2)} ${height_to_wheel}" rpy="0 0 0"/>
       <axis xyz="0 1 0"/>
     </joint>

File: description/urdf/plugins.gazebo.xacro (robot description, xacro)
@@ -3,5 +3,4 @@
     <!-- Constants -->
     <xacro:include filename="$(find description)/urdf/constants.xacro"/>
-<<<<<<< HEAD
     <!-- LIDAR -->
     <gazebo reference="scan_link">
@@ -37,5 +36,4 @@
         </sensor>
     </gazebo>
-=======
     <!-- Differential Drive Controller -->
     <gazebo>
@@ -71,4 +69,3 @@
         <plugin name="gazebo_ros_control" filename="libgazebo_ros_control.so"/>
     </gazebo>
->>>>>>> ef480fefc5cff283bff453b3ec6b471e0fc543b3
 </robot>

Commit message: fixed rviz

File: description/urdf/photon.urdf.xacro (robot description, xacro)
@@ -4,69 +4,48 @@
 Robot model taken from http://wiki.ros.org/pr2_mechanism/Tutorials/SImple%20URDF-Controller%20Example
 -->
-  <!-- Includes -->
-  <xacro:include filename="$(find description)/urdf/constants.xacro"/>
-  <xacro:include filename="$(find description)/urdf/inertias.xacro"/>
-  <xacro:include filename="$(find description)/urdf/photon_wheels.urdf.xacro"/>
-  <xacro:property name="deg_to_rad" value="0.01745329251994329577"/>
-  <!-- Constants for robot dimensions -->
-  <xacro:property name="axel_offset" value="0.05" /> <!-- Space btw top of beam and the each joint -->
-  <xacro:property name="steer_offset" value="0.02" /> <!-- Link 1 -->
-  <!-- Links: inertial,visual,collision -->
-  <link name="base_link">
-    <visual>
-      <origin xyz="0 0 0" rpy="0 0 0"/>
-      <geometry>
-        <mesh filename="$(find description)/urdf/meshes/StampedeBodyfxorigin.STL" scale="0.001 0.001 0.001"/>
-      </geometry>
-    </visual>
-    <collision>
-      <origin xyz="0 0 0" rpy="0 0 0"/>
-      <geometry>
-        <mesh filename="$(find description)/urdf/meshes/StampedeBodyfxorigin.STL" scale="0.001 0.001 0.001"/>
-      </geometry>
-    </collision>
-    <inertial>
-      <xacro:body_inertia/>
-    </inertial>
-  </link>
-  <link name="base_footprint">
-    <visual>
-      <geometry>
-        <sphere radius="0.01"/>
-      </geometry>
-    </visual>
-    <collision>
-      <origin xyz="0 0 0"/>
-      <geometry>
-        <sphere radius="0.00000001"/>
-      </geometry>
-    </collision>
-  </link>
-  <joint name="base_footprint_joint" type="fixed">
-    <origin xyz="0 0 ${wheel_radius}" rpy="0 0 0"/>
-    <child link="base_link"/>
-    <parent link="base_footprint"/>
-  </joint>
-  <!-- joints for ackermann_steering_controller -->
-  <xacro:front_steer name="front" parent="base" length="${fb_separation}"
-    steer_height="${wheel_radius+steer_offset}"/>
-  <xacro:rear_wheel name="rear" parent="base">
-    <origin xyz="${-fb_separation/2} 0 ${height_to_wheel}" rpy="${-90 * deg_to_rad} 0 0"/>
-  </xacro:rear_wheel>
-  <!-- Wheels -->
-  <xacro:front_wheel_lr name="front_right" parent="base" length="${fb_separation}"
-      width="${lr_separation}" right_left="1" steer_height="${wheel_radius+steer_offset}"/>
-  <xacro:front_wheel_lr name="front_left" parent="base" length="${fb_separation}"
-      width="${lr_separation}" right_left="-1" steer_height="${wheel_radius+steer_offset}"/>
-  <xacro:rear_wheel_lr name="rear_right" parent="base" length="${fb_separation}"
-      width="${lr_separation}" right_left="1"/>
-  <xacro:rear_wheel_lr name="rear_left" parent="base" length="${fb_separation}"
-      width="${lr_separation}" right_left="-1"/>
-  <!-- Colour -->
-  <gazebo reference="base_link">
-    <material>Gazebo/Green</material>
-  </gazebo>
-  <gazebo reference="base_footprint">
-    <material>Gazebo/Purple</material>
-  </gazebo>
+    <!-- Includes -->
+    <xacro:include filename="$(find description)/urdf/constants.xacro"/>
+    <xacro:include filename="$(find description)/urdf/inertias.xacro"/>
+    <xacro:include filename="$(find description)/urdf/photon_wheels.urdf.xacro"/>
+    <xacro:property name="deg_to_rad" value="0.01745329251994329577"/>
+    <!-- Constants for robot dimensions -->
+    <xacro:property name="axel_offset" value="0.05" /> <!-- Space btw top of beam and the each joint -->
+    <xacro:property name="steer_offset" value="0.02" /> <!-- Link 1 -->
+    <!-- Links: inertial,visual,collision -->
+    <link name="base_link">
+        <visual>
+        <origin xyz="0 0 0" rpy="0 0 0"/>
+        <geometry>
+            <mesh filename="package://description/urdf/meshes/Body.STL" scale="0.001 0.001 0.001"/>
+        </geometry>
+        </visual>
+        <collision>
+        <origin xyz="0 0 0" rpy="0 0 0"/>
+        <geometry>
+            <mesh filename="package://description/urdf/meshes/Body.STL" scale="0.001 0.001 0.001"/>
+        </geometry>
+        </collision>
+        <inertial>
+        <xacro:body_inertia/>
+        </inertial>
+    </link>
+    <!-- joints for ackermann_steering_controller -->
+    <xacro:front_steer name="front" parent="base" length="${fb_separation}"
+        steer_height="${wheel_radius+steer_offset}"/>
+    <xacro:rear_wheel name="rear" parent="base">
+        <origin xyz="${-fb_separation/2} 0 ${height_to_wheel}" rpy="${-90 * deg_to_rad} 0 0"/>
+    </xacro:rear_wheel>
+    <!-- Wheels -->
+    <xacro:front_wheel_lr name="front_right" parent="base" length="${fb_separation}"
+        width="${lr_separation}" right_left="1" steer_height="${wheel_radius+steer_offset}"/>
+    <xacro:front_wheel_lr name="front_left" parent="base" length="${fb_separation}"
+        width="${lr_separation}" right_left="-1" steer_height="${wheel_radius+steer_offset}"/>
+    <xacro:rear_wheel_lr name="rear_right" parent="base" length="${fb_separation}"
+        width="${lr_separation}" right_left="1"/>
+    <xacro:rear_wheel_lr name="rear_left" parent="base" length="${fb_separation}"
+        width="${lr_separation}" right_left="-1"/>
+    <!-- Colour -->
+    <gazebo reference="base_link">
+        <material>Gazebo/Green</material>
+    </gazebo>
 </robot>

File: description/urdf/photon_wheels.urdf.xacro (robot description, xacro)
@@ -76,5 +76,5 @@
         <origin xyz="0 0 0" rpy="0 0 0"/>
         <geometry>
-          <mesh filename="package://description/urdf/meshes/Wheelfxorigin.STL" scale="0.001 0.001 0.001"/>
+          <mesh filename="package://description/urdf/meshes/Wheels.STL" scale="0.001 0.001 0.001"/>
         </geometry>
       </visual>
@@ -82,5 +82,5 @@
         <origin xyz="0 0 0" rpy="0 0 0"/>
         <geometry>
-          <mesh filename="package://description/urdf/meshes/Wheelfxorigin.STL" scale="0.001 0.001 0.001"/>
+          <mesh filename="package://description/urdf/meshes/Wheels.STL" scale="0.001 0.001 0.001"/>
         </geometry>
       </collision>
@@ -157,5 +157,5 @@
         <origin xyz="0 0 0" rpy="0 0 0"/>
         <geometry>
-          <mesh filename="package://description/urdf/meshes/Wheelfxorigin.STL" scale="0.001 0.001 0.001"/>
+          <mesh filename="package://description/urdf/meshes/Wheels.STL" scale="0.001 0.001 0.001"/>
         </geometry>
       </visual>
@@ -163,5 +163,5 @@
         <origin xyz="0 0 0" rpy="0 0 0"/>
         <geometry>
-          <mesh filename="package://description/urdf/meshes/Wheelfxorigin.STL" scale="0.001 0.001 0.001"/>
+          <mesh filename="package://description/urdf/meshes/Wheels.STL" scale="0.001 0.001 0.001"/>
         </geometry>
       </collision>

Commit message: Small stylistic changes

File: description/urdf/photon.urdf.xacro (robot description, xacro)
@@ -28,5 +28,5 @@
         <parent link="base_link"/>
         <child link="body_link"/>
-        <origin xyz="0 0 0.0" rpy="0 0 0"/>
+        <origin xyz="0 0 0" rpy="0 0 0"/>
     </joint>
     <!-- Wheels -->
